Commit message: create robot model discription

File: robot_description/urdf/robot_mesh.urdf (robot description, URDF)
Before this commit: robot robot, 4 links, 3 joints
Links:
- link link_chassis: geometry collision mesh filename=package://robot_description/meshes/chassis.stl; visual mesh filename=package://robot_description/meshes/chassis.stl
- link link_left_wheel: geometry collision cylinder length=0.12 radius=0.08; collision cylinder length=0.12 radius=0.4
- link link_right_wheel: geometry collision cylinder length=0.12 radius=0.08; collision cylinder length=0.12 radius=0.4
